Commit message: ROS2, MIS

File: Sem4/ROS/install/irb120_ros2_gazebo/share/irb120_ros2_gazebo/urdf/abb_resources/common_materials.xacro (robot description, xacro)
@@ -77,3 +77,9 @@
     </material>
   </xacro:macro>
+  <xacro:macro name="inertial_rectangle" params="mass length width height">
+  <inertial>
+    <mass value="${mass}" />
+    <inertia ixx="${mass*(width^2 + height^2)/12}" ixy="0.0" ixz="0.0" iyy="${mass*(length^2 + height^2)/12}" iyz="0.0" izz="${mass*(length^2 + width^2)/12}" />
+  </inertial>
+</xacro:macro>
 </robot>

File: Sem4/ROS/install/irb120_ros2_gazebo/share/irb120_ros2_gazebo/urdf/irb120.urdf.xacro (robot description, xacro)
@@ -48,4 +48,99 @@
 -->
 <robot name="irb120" xmlns:xacro="http://ros.org/wiki/xacro">
+    <joint name="laser_joint" type="fixed">
+        <parent link="base_link"/>
+        <child link="laser_frame"/>
+        <origin xyz="0.1 0 0.2" rpy="0 0 0"/>
+    </joint>
+    <link name="laser_frame">
+        <visual>
+            <geometry>
+                <box size="0.01 0.01 0.01"/>
+            </geometry>
+            <material name="bblack"/>
+        </visual>
+        <collision>
+            <geometry>
+                <box size="0.01 0.01 0.01"/>
+            </geometry>
+        </collision>
+    </link>
+  <gazebo reference="laser_frame">
+      <material>Gazebo/Red</material>
+      <sensor name="laser" type="ray">
+          <pose> 0 0 0 0 0 0 </pose>
+          <visualize>true</visualize>
+          <update_rate>10</update_rate>
+          <ray>
+              <scan>
+                  <horizontal>
+                      <samples>360</samples>
+                      <min_angle>-3.14</min_angle>
+                      <max_angle>3.14</max_angle>
+                  </horizontal>
+              </scan>
+              <range>
+                  <min>0.3</min>
+                  <max>12</max>
+              </range>
+          </ray>
+          <plugin name="laser_controller" filename="libgazebo_ros_ray_sensor.so">
+              <ros>
+                  <argument>~/out:=scan</argument>
+              </ros>
+              <output_type>sensor_msgs/LaserScan</output_type>
+              <frame_name>laser_frame</frame_name>
+          </plugin>
+      </sensor>
+    </gazebo>
+    <joint name="camera_joint" type="fixed">
+        <parent link="base_link"/>
+        <child link="camera_link"/>
+        <origin xyz="0.5 0 0.99" rpy="0 -5 0"/>
+    </joint>
+    <link name="camera_link">
+        <visual>
+            <geometry>
+                <box size="0.010 0.03 0.03"/>
+            </geometry>
+            <material name="black"/>
+        </visual>
+        <visual>
+            <origin xyz="0 0 -0.05"/>
+            <geometry>
+                <cylinder radius="0.002" length="0.1"/>
+            </geometry>
+            <material name="black"/>
+        </visual>
+    </link>
+    <joint name="camera_optical_joint" type="fixed">
+        <parent link="camera_link"/>
+        <child link="camera_link_optical"/>
+        <origin xyz="0 0 0" rpy="${-pi/2} 0 ${-pi/2}"/>
+    </joint>
+    <link name="camera_link_optical"></link>
+    <gazebo reference="camera_link">
+        <material>Gazebo/Black</material>
+        <sensor name="camera" type="camera">
+            <pose> 0 0 0 0 0 0 </pose>
+            <visualize>true</visualize>
+            <update_rate>10</update_rate>
+            <camera>
+                <horizontal_fov>1.089</horizontal_fov>
+                <image>
+                    <format>R8G8B8</format>
+                    <width>640</width>
+                    <height>480</height>
+                </image>
+                <clip>
+                    <near>0.05</near>
+                    <far>8.0</far>
+                </clip>
+            </camera>
+            <plugin name="camera_controller" filename="libgazebo_ros_camera.so">
+                <frame_name>camera_link_optical</frame_name>
+            </plugin>
+        </sensor>
+    </gazebo>
   <!-- ===== ARGUMENTS ===== -->
   <!-- CELL LAYOUT:  -->

File: Sem4/ROS/install/irb120_ros2_gazebo/share/irb120_ros2_gazebo/urdf/irb120_transmission.xacro (robot description, xacro)
@@ -127,5 +127,4 @@
     </xacro:if>
     <!-- === SCHUNK EGP-64 GRIPPER === -->
-    <!-- ========== IR Reciver ========== -->
   </xacro:macro>
 </robot>
